File: Solar-Wing.sch (KiCad schematic (older format))
At the start: 3 parts

Commit message: Added footprint for XJT Prime solar cell
Parts:
- SC1, SC2, SC3: footprint (none) -> Solar-Wing:XTJ Prime
Changed lines of the file:
@@
 F 0 "SC1" V 3895 4050 50  0000 C CNN
 F 1 "Solar_Cell" V 3804 4050 50  0000 C CNN
-F 2 "" V 3650 4060 50  0001 C CNN
+F 2 "Solar-Wing:XTJ Prime" V 3650 4060 50  0001 C CNN
 F 3 "https://www.spectrolab.com/photovoltaics/XTJ-Prime_Data_Sheet.pdf" V 3650 4060 50  0001 C CNN
 	1    3650 4000
@@
 F 0 "SC2" V 4545 4050 50  0000 C CNN
 F 1 "Solar_Cell" V 4454 4050 50  0000 C CNN
-F 2 "" V 4300 4060 50  0001 C CNN
+F 2 "Solar-Wing:XTJ Prime" V 4300 4060 50  0001 C CNN
 F 3 "https://www.spectrolab.com/photovoltaics/XTJ-Prime_Data_Sheet.pdf" V 4300 4060 50  0001 C CNN
 	1    4300 4000
@@
 F 0 "SC3" V 5195 4050 50  0000 C CNN
 F 1 "Solar_Cell" V 5104 4050 50  0000 C CNN
-F 2 "" V 4950 4060 50  0001 C CNN
+F 2 "Solar-Wing:XTJ Prime" V 4950 4060 50  0001 C CNN
 F 3 "https://www.spectrolab.com/photovoltaics/XTJ-Prime_Data_Sheet.pdf" V 4950 4060 50  0001 C CNN
 	1    4950 4000

Commit message: PCB V1
Parts:
- added SC4: Solar_Cell, Solar-Wing:XTJ Prime, symbol Device:Solar_Cell
Connections:
- net +: now also SC4.1 (+)
- net -: now also SC4.2 (-)
Changed lines of the file:
@@
 	3750 3250 3750 4000
 Connection ~ 4400 3250
-Text GLabel 5400 3250 2    50   Input ~ 0
+Text GLabel 6400 3250 2    50   Input ~ 0
 -
+$Comp
+L Device:Solar_Cell SC4
+U 1 1 5EC9788E
+P 5550 4000
+F 0 "SC4" V 5795 4050 50  0000 C CNN
+F 1 "Solar_Cell" V 5704 4050 50  0000 C CNN
+F 2 "Solar-Wing:XTJ Prime" V 5550 4060 50  0001 C CNN
+F 3 "https://www.spectrolab.com/photovoltaics/XTJ-Prime_Data_Sheet.pdf" V 5550 4060 50  0001 C CNN
+	1    5550 4000
+	0    -1   -1   0
+$EndComp
 Wire Wire Line
-	5050 3250 5400 3250
+	5650 4000 6000 4000
+Wire Wire Line
+	6000 4000 6000 3250
+Wire Wire Line
+	6000 3250 6400 3250
+Wire Wire Line
+	5050 3250 6000 3250
 Connection ~ 5050 3250
+Connection ~ 6000 3250
+Wire Wire Line
+	5350 4000 5200 4000
+Wire Wire Line
+	5200 4000 5200 4400
+Wire Wire Line
+	5200 4400 4750 4400
+Connection ~ 4750 4400
 $EndSCHEMATC
